Commit message: Feat: make robot model generic with robot_name and robot_color parameters for multi-robot simulation

File: xacro/barista_robot_model.urdf.xacro (robot description, xacro)
@@ -1,118 +1,128 @@
 <?xml version="1.0"?>
-<robot xmlns:xacro="http://www.ros.org/wiki/xacro" name="barista_robot">
-    <!-- Arguments & Properties -->
-    <xacro:arg name="include_laser" default="true" />
-    <!-- Includes -->
-    <xacro:include filename="$(find barista_robot_description)/xacro/materials.xacro" />
-    <xacro:include filename="$(find barista_robot_description)/xacro/drive_wheel.xacro" />
-    <xacro:include filename="$(find barista_robot_description)/xacro/caster_wheel.xacro" />
-    <xacro:include filename="$(find barista_robot_description)/xacro/standoff_rod.xacro" />
-    <xacro:include filename="$(find barista_robot_description)/xacro/cup_holder_tray.xacro" />
-    <xacro:if value="$(arg include_laser)">
-        <xacro:include filename="$(find barista_robot_description)/xacro/laser_scanner.xacro" />
-    </xacro:if>
-    <link name="base_footprint"/>
-    <!-- Main Body-->
-    <link name="base_link">
-        <visual>
-            <geometry>
-                <cylinder length="0.155" radius="0.178"/>
-            </geometry>
-            <material name="red"/>
-        </visual>
-        <collision>
-            <geometry>
-                <cylinder length="0.155" radius="0.178"/>
-            </geometry>
-        </collision>
-        <inertial>
-            <mass value="8.0"/>
-            <inertia ixx="0.07938466666666666" ixy="0" ixz="0" iyy="0.07938466666666666" iyz="0" izz="0.126736"/>
-        </inertial>
-    </link>
-    <gazebo reference="base_link">
-        <material>Gazebo/Red</material>
-    </gazebo>
-    <joint name="base_footprint_joint" type="fixed">
-        <origin xyz="0 0 0.1025" rpy="0 0 0" />  <!-- Clearance 0.025 + Body Height 0.0775-->
-        <parent link="base_footprint" />
-        <child link="base_link" />
-    </joint>
-    <!-- Wheel Left -->
-    <xacro:drive_wheel name="left_wheel" parent="base_link" xyz="0 0.15 -0.0673" />  <!-- 0.0352-0.1025-->
-    <!-- Wheel Right -->
-    <xacro:drive_wheel name="right_wheel" parent="base_link" xyz="0 -0.15 -0.0673" />
-    <!-- Front Caster Wheel -->
-    <xacro:caster_wheel name="front_caster" parent="base_link" xyz="0.15 0 -0.0775" />
-    <!-- Back Caster Wheel -->
-    <xacro:caster_wheel name="back_caster" parent="base_link" xyz="-0.15 0 -0.0775" />
-    <!-- Standoff Rods Left -->
-    <xacro:standoff_rod name="left_front_standoff_rod"
-        parent="base_link"
-        xyz="0.04 0.13 0.1875"
-        length="0.22"
-        radius="0.01"
-        />
-    <xacro:standoff_rod name="left_back_standoff_rod"
-        parent="base_link"
-        xyz="-0.04 0.13 0.1875"
-        length="0.22"
-        radius="0.01"
-        />
-    <!-- Standoff Rods Right-->
-    <xacro:standoff_rod name="right_front_standoff_rod"
-        parent="base_link"
-        xyz="0.04 -0.13 0.1875"
-        length="0.22"
-        radius="0.01"
-        />
-    <xacro:standoff_rod name="right_back_standoff_rod"
-        parent="base_link"
-        xyz="-0.04 -0.13 0.1875"
-        length="0.22"
-        radius="0.01"
-        />
-    <!-- Cup Holder Tray --> <!-- 0.0775 + 0.22 + 0.045-->
-    <xacro:cup_holder_tray name="cup_holder_tray" parent="base_link" xyz="0.0 0.0 0.3425" />
-    <!-- Planar Laser Scanner -->
-    <xacro:if value="$(arg include_laser)">
-        <xacro:laser_scanner name="laser_scan" parent="base_link" xyz="0.11 0.0 0.0775" />
-    </xacro:if>
-    <!-- PLUGINS -->
-    <!-- JOINT PUBLISHER -->
-    <gazebo>
-        <plugin name="barista_robot_joint_state" filename="libgazebo_ros_joint_state_publisher.so">
-            <ros>
-                <remapping>~/out:=joint_states</remapping>
-            </ros>
-            <update_rate>30</update_rate>
-            <joint_name>left_wheel_joint</joint_name>
-            <joint_name>right_wheel_joint</joint_name>
-            <joint_name>front_caster_yaw_joint</joint_name>
-            <joint_name>back_caster_yaw_joint</joint_name>
-            <joint_name>front_caster_roll_joint</joint_name>
-            <joint_name>back_caster_roll_joint</joint_name>
-            <joint_name>front_caster_pitch_joint</joint_name>
-            <joint_name>back_caster_pitch_joint</joint_name>
-        </plugin>
-    </gazebo>
-    <!-- Differential drive -->
-    <gazebo>
-        <plugin filename="libgazebo_ros_diff_drive.so" name="differential_drive_controller">
-            <!-- wheels -->
-            <left_joint>left_wheel_joint</left_joint>
-            <right_joint>right_wheel_joint</right_joint>
-            <!-- kinematics -->
-            <wheel_separation>0.3</wheel_separation>
-            <wheel_diameter>0.0704</wheel_diameter>
-            <!-- limits -->
-            <max_wheel_torque>10.0</max_wheel_torque>
-            <max_wheel_acceleration>2.0</max_wheel_acceleration>
-            <!-- output -->
-            <publish_odom>true</publish_odom>
-            <publish_odom_tf>true</publish_odom_tf>
-            <odometry_frame>odom</odometry_frame>
-            <robot_base_frame>base_footprint</robot_base_frame>
-        </plugin>
-    </gazebo>
+<robot xmlns:xacro="http://www.ros.org/wiki/xacro" name="${robot_name}">
+  <!-- Arguments & Properties -->
+  <xacro:arg name="robot_name" default="barista_robot"/>
+  <xacro:arg name="robot_color" default="red"/>
+  <xacro:arg name="include_laser" default="true"/>
+  <!-- Includes -->
+  <xacro:include filename="$(find barista_robot_description)/xacro/materials.xacro" />
+  <xacro:include filename="$(find barista_robot_description)/xacro/drive_wheel.xacro" />
+  <xacro:include filename="$(find barista_robot_description)/xacro/caster_wheel.xacro" />
+  <xacro:include filename="$(find barista_robot_description)/xacro/standoff_rod.xacro" />
+  <xacro:include filename="$(find barista_robot_description)/xacro/cup_holder_tray.xacro" />
+  <xacro:if value="$(arg include_laser)">
+    <xacro:include filename="$(find barista_robot_description)/xacro/laser_scanner.xacro" />
+  </xacro:if>
+  <!-- Base footprint (kept unprefixed inside model) -->
+  <link name="base_footprint"/>
+  <!-- Main Body-->
+  <link name="base_link">
+    <visual>
+      <geometry>
+        <cylinder length="0.155" radius="0.178"/>
+      </geometry>
+      <material name="${robot_color}"/>
+    </visual>
+    <collision>
+      <geometry>
+        <cylinder length="0.155" radius="0.178"/>
+      </geometry>
+    </collision>
+    <inertial>
+      <mass value="8.0"/>
+      <inertia ixx="0.07938466666666666" ixy="0" ixz="0"
+               iyy="0.07938466666666666" iyz="0" izz="0.126736"/>
+    </inertial>
+  </link>
+  <!-- Gazebo visual material (uses robot_color) -->
+  <gazebo reference="base_link">
+    <material>Gazebo/${robot_color}</material>
+  </gazebo>
+  <joint name="base_footprint_joint" type="fixed">
+    <origin xyz="0 0 0.1025" rpy="0 0 0" />
+    <parent link="base_footprint" />
+    <child link="base_link" />
+  </joint>
+  <!-- Wheel Left -->
+  <xacro:drive_wheel name="left_wheel" parent="base_link" xyz="0 0.15 -0.0673" />
+  <!-- Wheel Right -->
+  <xacro:drive_wheel name="right_wheel" parent="base_link" xyz="0 -0.15 -0.0673" />
+  <!-- Front Caster Wheel -->
+  <xacro:caster_wheel name="front_caster" parent="base_link" xyz="0.15 0 -0.0775" />
+  <!-- Back Caster Wheel -->
+  <xacro:caster_wheel name="back_caster" parent="base_link" xyz="-0.15 0 -0.0775" />
+  <!-- Standoff Rods Left -->
+  <xacro:standoff_rod name="left_front_standoff_rod"
+      parent="base_link"
+      xyz="0.04 0.13 0.1875"
+      length="0.22"
+      radius="0.01" />
+  <xacro:standoff_rod name="left_back_standoff_rod"
+      parent="base_link"
+      xyz="-0.04 0.13 0.1875"
+      length="0.22"
+      radius="0.01" />
+  <!-- Standoff Rods Right-->
+  <xacro:standoff_rod name="right_front_standoff_rod"
+      parent="base_link"
+      xyz="0.04 -0.13 0.1875"
+      length="0.22"
+      radius="0.01" />
+  <xacro:standoff_rod name="right_back_standoff_rod"
+      parent="base_link"
+      xyz="-0.04 -0.13 0.1875"
+      length="0.22"
+      radius="0.01" />
+  <!-- Cup Holder Tray -->
+  <!-- pass color argument to the macro so cup holder uses robot_color visually -->
+  <xacro:cup_holder_tray name="cup_holder_tray" parent="base_link" xyz="0.0 0.0 0.3425" color="${robot_color}" />
+  <!-- Planar Laser Scanner -->
+  <xacro:if value="$(arg include_laser)">
+    <!-- pass robot_name into laser xacro so the laser plugin can namespace topics -->
+    <xacro:laser_scanner name="laser_scan" parent="base_link" xyz="0.11 0.0 0.0775" robot_name="${robot_name}" />
+  </xacro:if>
+  <!-- PLUGINS -->
+  <!-- JOINT STATE PUBLISHER (namespaced) -->
+  <gazebo>
+    <plugin name="${robot_name}_joint_state" filename="libgazebo_ros_joint_state_publisher.so">
+      <ros>
+        <namespace>/${robot_name}</namespace>
+        <remapping>~/out:=joint_states</remapping>
+      </ros>
+      <update_rate>30</update_rate>
+      <!-- Note: joint names kept as defined in sub-xacro (no global prefix) -->
+      <joint_name>left_wheel_joint</joint_name>
+      <joint_name>right_wheel_joint</joint_name>
+      <joint_name>front_caster_yaw_joint</joint_name>
+      <joint_name>back_caster_yaw_joint</joint_name>
+      <joint_name>front_caster_roll_joint</joint_name>
+      <joint_name>back_caster_roll_joint</joint_name>
+      <joint_name>front_caster_pitch_joint</joint_name>
+      <joint_name>back_caster_pitch_joint</joint_name>
+    </plugin>
+  </gazebo>
+  <!-- Differential drive (namespaced) -->
+  <gazebo>
+    <plugin filename="libgazebo_ros_diff_drive.so" name="${robot_name}_differential_drive">
+      <ros>
+        <namespace>/${robot_name}</namespace>
+        <remapping>/cmd_vel:=cmd_vel</remapping>
+      </ros>
+      <!-- wheels -->
+      <left_joint>left_wheel_joint</left_joint>
+      <right_joint>right_wheel_joint</right_joint>
+      <!-- kinematics -->
+      <wheel_separation>0.3</wheel_separation>
+      <wheel_diameter>0.0704</wheel_diameter>
+      <!-- limits -->
+      <max_wheel_torque>10.0</max_wheel_torque>
+      <max_wheel_acceleration>2.0</max_wheel_acceleration>
+      <!-- output -->
+      <publish_odom>true</publish_odom>
+      <publish_odom_tf>true</publish_odom_tf>
+      <!-- keep frame ids local (launch can add frame_prefix if desired) -->
+      <odometry_frame>odom</odometry_frame>
+      <robot_base_frame>base_footprint</robot_base_frame>
+    </plugin>
+  </gazebo>
 </robot>

File: xacro/cup_holder_tray.xacro (robot description, xacro)
@@ -1,38 +1,41 @@
 <?xml version="1.0"?>
 <robot xmlns:xacro="http://www.ros.org/wiki/xacro">
-    <xacro:property name="cup_holder_mass" value="1.0" />
-    <xacro:property name="cup_holder_radius" value="0.16" />
-    <xacro:property name="cup_holder_length" value="0.09" />
-    <!-- Cup Holder Tray Wheel Macro -->
-    <xacro:macro name="cup_holder_tray" params="name parent xyz">
-       <link name="${name}">
-            <visual>
-                <geometry>
-                    <cylinder length="${cup_holder_length}" radius="${cup_holder_radius}"/>
-                </geometry>
-                <material name="red"/>
-            </visual>
-            <collision>
-                <geometry>
-                    <cylinder length="${cup_holder_length}" radius="${cup_holder_radius}"/>
-                </geometry>
-            </collision>
-           <inertial>
-                <mass value="${cup_holder_mass}"/>
-                <inertia
-                    ixx="${(1.0/12.0)*cup_holder_mass*(3*cup_holder_radius*cup_holder_radius + cup_holder_length*cup_holder_length)}"
-                    ixy="0" ixz="0"
-                    iyy="${(1.0/12.0)*cup_holder_mass*(3*cup_holder_radius*cup_holder_radius + cup_holder_length*cup_holder_length)}" iyz="0"
-                    izz="${(1.0/2.0)*cup_holder_mass*cup_holder_radius*cup_holder_radius}"/>
-            </inertial>
-        </link>
-        <gazebo reference="${name}">
-            <material>Gazebo/Red</material>
-        </gazebo>
-        <joint name="${name}_joint" type="fixed">
-            <origin xyz="${xyz}" rpy="0 0 0" />
-            <parent link="${parent}" />
-            <child link="${name}" />
-        </joint>
-    </xacro:macro>
+  <xacro:property name="cup_holder_mass" value="1.0" />
+  <xacro:property name="cup_holder_radius" value="0.16" />
+  <xacro:property name="cup_holder_length" value="0.09" />
+  <!-- Cup Holder Tray Macro -->
+  <xacro:macro name="cup_holder_tray" params="name parent xyz color">
+    <link name="${name}">
+      <visual>
+        <geometry>
+          <cylinder length="${cup_holder_length}" radius="${cup_holder_radius}"/>
+        </geometry>
+        <material name="${color}"/>
+      </visual>
+      <collision>
+        <geometry>
+          <cylinder length="${cup_holder_length}" radius="${cup_holder_radius}"/>
+        </geometry>
+      </collision>
+      <inertial>
+        <mass value="${cup_holder_mass}"/>
+        <inertia
+          ixx="${(1.0/12.0)*cup_holder_mass*(3*cup_holder_radius*cup_holder_radius + cup_holder_length*cup_holder_length)}"
+          ixy="0" ixz="0"
+          iyy="${(1.0/12.0)*cup_holder_mass*(3*cup_holder_radius*cup_holder_radius + cup_holder_length*cup_holder_length)}"
+          iyz="0"
+          izz="${(1.0/2.0)*cup_holder_mass*cup_holder_radius*cup_holder_radius}"/>
+      </inertial>
+    </link>
+    <!-- Gazebo visual color -->
+    <gazebo reference="${name}">
+      <material>Gazebo/${color}</material>
+    </gazebo>
+    <!-- Fixed joint -->
+    <joint name="${name}_joint" type="fixed">
+      <origin xyz="${xyz}" rpy="0 0 0" />
+      <parent link="${parent}" />
+      <child link="${name}" />
+    </joint>
+  </xacro:macro>
 </robot>

File: xacro/laser_scanner.xacro (robot description, xacro)
@@ -1,83 +1,81 @@
 <?xml version="1.0"?>
 <robot xmlns:xacro="http://www.ros.org/wiki/xacro">
-    <xacro:property name="laser_scan_length" value="0.05"/>
-    <xacro:property name="laser_scan_width" value="0.05"/>
-    <xacro:property name="laser_scan_height" value="0.07"/>
-    <xacro:property name="laser_scan_mass" value="0.13" />
-    <xacro:macro name="laser_scanner" params="name parent xyz">
-        <link name="${name}">
-            <visual>
-                <geometry>
-                    <mesh filename="package://barista_robot_description/meshes/hokuyo_ust_10lx.dae" scale="1.0 1.0 1.0"/>
-                </geometry>
-            </visual>
-            <collision>
-                <origin xyz="0 0 ${laser_scan_height/2}" rpy="0 0 0"/>
-                <geometry>
-                    <box size="${laser_scan_length} ${laser_scan_width} ${laser_scan_height}"/>
-                </geometry>
-            </collision>
-            <inertial>
-                <origin xyz="0 0 ${laser_scan_height/2}" rpy="0 0 0"/>
-                <mass value="${laser_scan_mass}"/>
-                <inertia
-                    ixx="${(1.0/12.0)*laser_scan_mass*(laser_scan_width*laser_scan_width + laser_scan_height*laser_scan_height)}"
-                    ixy="0" ixz="0"
-                    iyy="${(1.0/12.0)*laser_scan_mass*(laser_scan_length*laser_scan_length + laser_scan_height*laser_scan_height)}" iyz="0"
-                    izz="${(1.0/12.0)*laser_scan_mass*(laser_scan_length*laser_scan_length + laser_scan_width*laser_scan_width)}"/>
-            </inertial>
-        </link>
-        <joint name="${name}_joint" type="fixed">
-            <origin xyz="${xyz}" rpy="0 0 0" />
-            <parent link="${parent}"/>
-            <child link="${name}"/>
-        </joint>
-        <link name="${name}_frame">
-        </link>
-        <joint name="${name}_frame_joint" type="fixed">
-            <origin xyz="0.025 0 0.05" rpy="0 0 0" />
-            <parent link="${name}"/>
-            <child link="${name}_frame"/>
-        </joint>
-        <gazebo reference="${name}_frame">
-            <sensor name="${name}_sensor" type="ray">
-                <pose>0 0 0 0 0 0</pose>
-                <always_on>true</always_on>
-                <visualize>true</visualize>
-                <update_rate>100.0</update_rate>
-                <ray>
-                    <scan>
-                        <horizontal>
-                            <samples>720</samples>
-                            <resolution>1.0</resolution>
-                            <min_angle>-3.14</min_angle>
-                            <max_angle>3.14</max_angle>
-                        </horizontal>
-                        <vertical>
-                            <samples>1</samples>
-                            <resolution>1.0</resolution>
-                            <min_angle>0.0</min_angle>
-                            <max_angle>0.0</max_angle>
-                        </vertical>
-                    </scan>
-                    <range>
-                        <min>0.1</min>
-                        <max>10.0</max>
-                    </range>
-                    <!-- <noise>
-                        <type>gaussian</type>
-                        <mean>0.0</mean>
-                        <stddev>0.01</stddev>
-                    </noise> -->
-                </ray>
-                <plugin name="laser" filename="libgazebo_ros_ray_sensor.so">
-                    <ros>
-                        <remapping>~/out:=scan</remapping>
-                    </ros>
-                    <output_type>sensor_msgs/LaserScan</output_type>
-                    <frame_name>${name}_frame</frame_name>
-                </plugin>
-            </sensor>
-	    </gazebo>
-    </xacro:macro>
+  <xacro:property name="laser_scan_length" value="0.05"/>
+  <xacro:property name="laser_scan_width" value="0.05"/>
+  <xacro:property name="laser_scan_height" value="0.07"/>
+  <xacro:property name="laser_scan_mass" value="0.13"/>
+  <!-- Laser Scanner Macro -->
+  <xacro:macro name="laser_scanner" params="name parent xyz robot_name">
+    <link name="${name}">
+      <visual>
+        <geometry>
+          <mesh filename="package://barista_robot_description/meshes/hokuyo_ust_10lx.dae" scale="1.0 1.0 1.0"/>
+        </geometry>
+      </visual>
+      <collision>
+        <origin xyz="0 0 ${laser_scan_height/2}" rpy="0 0 0"/>
+        <geometry>
+          <box size="${laser_scan_length} ${laser_scan_width} ${laser_scan_height}"/>
+        </geometry>
+      </collision>
+      <inertial>
+        <origin xyz="0 0 ${laser_scan_height/2}" rpy="0 0 0"/>
+        <mass value="${laser_scan_mass}"/>
+        <inertia
+          ixx="${(1.0/12.0)*laser_scan_mass*(laser_scan_width*laser_scan_width + laser_scan_height*laser_scan_height)}"
+          ixy="0" ixz="0"
+          iyy="${(1.0/12.0)*laser_scan_mass*(laser_scan_length*laser_scan_length + laser_scan_height*laser_scan_height)}"
+          iyz="0"
+          izz="${(1.0/12.0)*laser_scan_mass*(laser_scan_length*laser_scan_length + laser_scan_width*laser_scan_width)}"/>
+      </inertial>
+    </link>
+    <joint name="${name}_joint" type="fixed">
+      <origin xyz="${xyz}" rpy="0 0 0" />
+      <parent link="${parent}"/>
+      <child link="${name}"/>
+    </joint>
+    <link name="${name}_frame" />
+    <joint name="${name}_frame_joint" type="fixed">
+      <origin xyz="0.025 0 0.05" rpy="0 0 0" />
+      <parent link="${name}"/>
+      <child link="${name}_frame"/>
+    </joint>
+    <!-- Gazebo sensor plugin -->
+    <gazebo reference="${name}_frame">
+      <sensor name="${name}_sensor" type="ray">
+        <pose>0 0 0 0 0 0</pose>
+        <always_on>true</always_on>
+        <visualize>true</visualize>
+        <update_rate>100.0</update_rate>
+        <ray>
+          <scan>
+            <horizontal>
+              <samples>720</samples>
+              <resolution>1.0</resolution>
+              <min_angle>-3.14</min_angle>
+              <max_angle>3.14</max_angle>
+            </horizontal>
+            <vertical>
+              <samples>1</samples>
+              <resolution>1.0</resolution>
+              <min_angle>0.0</min_angle>
+              <max_angle>0.0</max_angle>
+            </vertical>
+          </scan>
+          <range>
+            <min>0.1</min>
+            <max>10.0</max>
+          </range>
+        </ray>
+        <plugin name="${robot_name}_laser" filename="libgazebo_ros_ray_sensor.so">
+          <ros>
+            <namespace>/${robot_name}</namespace>
+            <remapping>~/out:=scan</remapping>
+          </ros>
+          <output_type>sensor_msgs/LaserScan</output_type>
+          <frame_name>${name}_frame</frame_name>
+        </plugin>
+      </sensor>
+    </gazebo>
+  </xacro:macro>
 </robot>
